Commit message: Add TouchSensor to FencingSwordAsSlot for contact detection and refactoring code for readability

File: controllers/combot_controller/combot_urdf.urdf (robot description, URDF)
Before this commit: robot ComBot, 91 links, 90 joints
Links:
- removed link Hokuyo URG-04LX-UG01
- removed link cap screw(1)_23
- removed link cap screw(10)_14
- removed link cap screw(11)_13
- removed link cap screw(12)_12
- removed link cap screw(13)_11
- removed link cap screw(14)_10
- removed link cap screw(15)_9
- removed link cap screw(16)_8
- removed link cap screw(17)_7
- removed link cap screw(18)_6
- removed link cap screw(19)_5
- removed link cap screw(2)_22
- removed link cap screw(3)_21
- removed link cap screw(4)_20
- removed link cap screw(5)_19
- removed link cap screw(6)_18
- removed link cap screw(7)_17
- removed link cap screw(8)_16
- removed link cap screw(9)_15
- removed link cap screw_24
- removed link gripper_left_finger_link_4
- removed link gripper_right_finger_link_3
- added link Velodyne VLP-16; collision cylinder length=0.0727 radius=0.052; visual cylinder length=0.0727 radius=0.052
- added link sword_tip_sensor; collision sphere radius=0.03; visual sphere radius=0.03
- link right: geometry collision cylinder length=0.67 radius=0.04; collision sphere radius=0.04
Joints:
- removed joint base_link_Hokuyo URG-04LX-UG01_joint
- removed joint right_cap screw(1)_23_joint
- removed joint right_cap screw(10)_14_joint
- removed joint right_cap screw(11)_13_joint
- removed joint right_cap screw(12)_12_joint
- removed joint right_cap screw(13)_11_joint
- removed joint right_cap screw(14)_10_joint
- removed joint right_cap screw(15)_9_joint
- removed joint right_cap screw(16)_8_joint
- removed joint right_cap screw(17)_7_joint
- removed joint right_cap screw(18)_6_joint
- removed joint right_cap screw(19)_5_joint
- removed joint right_cap screw(2)_22_joint
- removed joint right_cap screw(3)_21_joint
- removed joint right_cap screw(4)_20_joint
- removed joint right_cap screw(5)_19_joint
- removed joint right_cap screw(6)_18_joint
- removed joint right_cap screw(7)_17_joint
- removed joint right_cap screw(8)_16_joint
- removed joint right_cap screw(9)_15_joint
- removed joint right_cap screw_24_joint
- removed joint right_hand_gripper_left_finger_joint
- removed joint right_hand_gripper_right_finger_joint
- added joint base_link_Velodyne VLP-16_joint: type fixed, parent base_link, child Velodyne VLP-16, origin xyz=-0.208 0 0.236 rpy=0 0 0
- added joint right_sword_tip_sensor_joint: type fixed, parent right, child sword_tip_sensor, origin xyz=0 0.56 0.06 rpy=0 0 0
- joint left_cap screw(19)_joint: origin xyz=0.0815 -0.002896 -0.0004 rpy=3.14159 0 0 -> xyz=0.0415 -0.0029 -0.0004 rpy=3.14159 0 0
- joint left_hand_gripper_left_finger_joint: origin xyz=0.04 0 0 rpy=0 0 3.1415 -> xyz=0 0 0 rpy=0 0 3.1415
- joint torso_lift_joint: limit lower=0 upper=0.35 effort=2000 velocity=0.07 -> lower=0 upper=0.35 effort=2000 velocity=0.2
- joint wrist_right_ft_tool_link_right_joint: origin xyz=0.016 0 0 rpy=-2.356193 1.570792 0.785393 -> xyz=0.2 -0.000001 -0.05 rpy=0 0 -1.5708
